File: Hardware/BLDC_Motor_Driver/MCU.kicad_sch (KiCad schematic)
At the start: 0 parts

Commit message: started the MCU and Finializing the MCU the next step will be the DRV
Parts:
- added C1, C2, C3, C4, C5, C6: 0.1u, Capacitor_SMD:C_0805_2012Metric_Pad1.18x1.45mm_HandSolder, symbol Device:C
- added C10, C9: 12p, Capacitor_SMD:C_0805_2012Metric_Pad1.18x1.45mm_HandSolder, symbol Device:C
- added C7: 1u, Capacitor_SMD:C_0805_2012Metric_Pad1.18x1.45mm_HandSolder, symbol Device:C
- added C8: 4.7u, Capacitor_SMD:C_0805_2012Metric_Pad1.18x1.45mm_HandSolder, symbol Device:C
- added U1: STM32G431RBTx, Package_QFP:LQFP-64_10x10mm_P0.5mm, symbol MCU_ST_STM32G4:STM32G431RBTx
- added Y1: Crystal_GND24, symbol Device:Crystal_GND24
- added Y2: Crystal, symbol Device:Crystal
Connections:
- new net: C1.1, C2.1, C3.1, C5.1, C6.1, C7.1, C8.1, U1.1 (VBAT), U1.16 (VDD), U1.29 (VDDA), U1.32 (VDD), U1.48 (VDD), U1.64 (VDD)
- new net: C1.2, C2.2, C3.2, C5.2, C6.2, C7.2, C8.2
- new net: C9.2, U1.3 (PC14), Y2.2
- new net: C10.2, U1.4 (PC15), Y2.1
- new net: U1.5 (PF0), Y1.3
- new net: U1.6 (PF1), Y1.1
- new net +3.3V: C4.1
- new net GND: C10.1, C4.2, C9.1, U1.15 (VSS), U1.27 (VSSA), U1.31 (VSS), U1.47 (VSS), U1.63 (VSS), Y1.2, Y1.4
