File: Hardware/BLDC_MC_V1.0/BLDC_MC_V1.0_Voltage_Sensor.kicad_sch (KiCad schematic)
At the start: 28 parts, among them U12 TLV9061IDBVR, U13 TLV9061IDBVR, U14 TLV9061IDBVR, U15 TLV9061IDBVR

Commit message: Solve all errors and wornings in project
Other:
- title: BLDC_MC_V1.0_Voltage_Sensor -> ${Project_Name}
Changed lines of the file:
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@@
 	(paper "A4")
 	(title_block
-		(title "BLDC_MC_V1.0_Voltage_Sensor")
+		(title "${Project_Name}")
 		(date "2026-03-11")
 		(rev "V1")
@@
 			)
 		)
-		(property "Datasheet" "https://www.lcsc.com/datasheet/C28233.pdf"
+		(property "Datasheet" "~"
 			(at 144.78 173.99 0)
 			(effects
@@
 			)
 		)
-		(property "Datasheet" "https://www.lcsc.com/datasheet/C705760.pdf"
+		(property "Datasheet" "~"
 			(at 35.56 180.34 0)
 			(effects
@@
 			)
 		)
-		(property "Datasheet" "https://www.lcsc.com/datasheet/C28233.pdf"
+		(property "Datasheet" "~"
 			(at 144.78 60.96 0)
 			(effects
@@
 			)
 		)
-		(property "Datasheet" "https://www.lcsc.com/datasheet/C870633.pdf"
+		(property "Datasheet" "~"
 			(at 35.56 52.07 0)
 			(effects
@@
 			)
 		)
-		(property "Description" "2.7kΩ ±0.1% 250mW 1206 Thin Film Resistor"
+		(property "Description" "Resistor"
 			(at 35.56 52.07 0)
 			(effects
@@
 			)
 		)
-		(property "Datasheet" "https://www.lcsc.com/datasheet/C28233.pdf"
+		(property "Datasheet" "~"
 			(at 60.96 179.07 0)
 			(effects
@@
 			)
 		)
-		(property "Datasheet" "https://www.lcsc.com/datasheet/C28233.pdf"
+		(property "Datasheet" "~"
 			(at 176.53 67.31 0)
 			(effects
@@
 			)
 		)
-		(property "Datasheet" "https://www.lcsc.com/datasheet/C108661.pdf"
+		(property "Datasheet" "~"
 			(at 50.8 59.69 0)
 			(effects
@@
 			)
 		)
-		(property "Datasheet" "https://www.lcsc.com/datasheet/C95204.pdf"
+		(property "Datasheet" "~"
 			(at 165.1 66.04 0)
 			(effects
@@
 			)
 		)
-		(property "Datasheet" "https://www.lcsc.com/datasheet/C28233.pdf"
+		(property "Datasheet" "~"
 			(at 60.96 123.19 0)
 			(effects
@@
 			)
 		)
-		(property "Datasheet" "https://www.lcsc.com/datasheet/C705760.pdf"
+		(property "Datasheet" "~"
 			(at 35.56 68.58 0)
 			(effects
@@
 			)
 		)
-		(property "Datasheet" "https://www.lcsc.com/datasheet/C108661.pdf"
+		(property "Datasheet" "~"
 			(at 128.27 115.57 0)
 			(effects
@@
 			)
 		)
-		(property "Datasheet" "https://www.lcsc.com/datasheet/C108661.pdf"
+		(property "Datasheet" "~"
 			(at 50.8 171.45 0)
 			(effects
@@
 			)
 		)
-		(property "Datasheet" "https://www.lcsc.com/datasheet/C95204.pdf"
+		(property "Datasheet" "~"
 			(at 165.1 52.07 0)
 			(effects
@@
 			)
 		)
-		(property "Datasheet" "https://www.lcsc.com/datasheet/C28233.pdf"
+		(property "Datasheet" "~"
 			(at 266.7 64.77 0)
 			(effects
@@
 			)
 		)
-		(property "Datasheet" "https://www.lcsc.com/datasheet/C870633.pdf"
+		(property "Datasheet" "~"
 			(at 35.56 163.83 0)
 			(effects
@@
 			)
 		)
-		(property "Description" "2.7kΩ ±0.1% 250mW 1206 Thin Film Resistor"
+		(property "Description" "Resistor"
 			(at 35.56 163.83 0)
 			(effects
@@
 			)
 		)
-		(property "Datasheet" "https://www.lcsc.com/datasheet/C28233.pdf"
+		(property "Datasheet" "~"
 			(at 144.78 118.11 0)
 			(effects
@@
 			)
 		)
-		(property "Datasheet" "https://www.lcsc.com/datasheet/C108661.pdf"
+		(property "Datasheet" "~"
 			(at 128.27 59.69 0)
 			(effects
@@
 			)
 		)
-		(property "Datasheet" "https://www.lcsc.com/datasheet/C28233.pdf"
+		(property "Datasheet" "~"
 			(at 60.96 67.31 0)
 			(effects
@@
 			)
 		)
-		(property "Datasheet" "https://www.lcsc.com/datasheet/C51205.pdf"
+		(property "Datasheet" "~"
 			(at 189.23 67.31 0)
 			(effects
@@
 			)
 		)
-		(property "Datasheet" "https://www.lcsc.com/datasheet/C28233.pdf"
+		(property "Datasheet" "~"
 			(at 250.19 67.31 0)
 			(effects
@@
 			)
 		)
-		(property "Datasheet" "https://www.lcsc.com/datasheet/C705760.pdf"
+		(property "Datasheet" "~"
 			(at 35.56 124.46 0)
 			(effects
@@
 			)
 		)
-		(property "Datasheet" "https://www.lcsc.com/datasheet/C870633.pdf"
+		(property "Datasheet" "~"
 			(at 35.56 107.95 0)
 			(effects
@@
 			)
 		)
-		(property "Description" "2.7kΩ ±0.1% 250mW 1206 Thin Film Resistor"
+		(property "Description" "Resistor"
 			(at 35.56 107.95 0)
 			(effects
@@
 			)
 		)
-		(property "Datasheet" "https://www.lcsc.com/datasheet/C108661.pdf"
+		(property "Datasheet" "~"
 			(at 128.27 171.45 0)
 			(effects
@@
 			)
 		)
-		(property "Datasheet" "https://www.lcsc.com/datasheet/C108661.pdf"
+		(property "Datasheet" "~"
 			(at 50.8 115.57 0)
 			(effects
