File: Hardware/BLDC_MC_V1.0/BLDC_MC_V1.0_Voltage_Sensor.kicad_sch (KiCad schematic)
At the start: 28 parts, among them U12 TLV9061IDBVR, U13 TLV9061IDBVR, U14 TLV9061IDBVR, U15 TLV9061IDBVR

Commit message: Edited the MPN of the 100K resistor
Parts:
- R55, R58, R61: LCSC_PN C870633 -> C2907368; MP RT1206BRD072K7L -> FRC1206F1003TS
- R56, R59, R62: value 2k6 -> 2k7
Changed lines of the file:
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@@
 			)
 		)
-		(property "Value" "2k6"
+		(property "Value" "2k7"
 			(at 38.1 181.6099 0)
 			(show_name no)
@@
 			)
 		)
-		(property "LCSC_PN" "C870633"
+		(property "LCSC_PN" "C2907368"
 			(at 35.56 52.07 0)
 			(hide yes)
@@
 			)
 		)
-		(property "MP" "RT1206BRD072K7L"
+		(property "MP" "FRC1206F1003TS"
 			(at 35.56 52.07 0)
 			(hide yes)
@@
 			)
 		)
-		(property "Value" "2k6"
+		(property "Value" "2k7"
 			(at 38.1 69.8499 0)
 			(show_name no)
@@
 			)
 		)
-		(property "LCSC_PN" "C870633"
+		(property "LCSC_PN" "C2907368"
 			(at 35.56 163.83 0)
 			(hide yes)
@@
 			)
 		)
-		(property "MP" "RT1206BRD072K7L"
+		(property "MP" "FRC1206F1003TS"
 			(at 35.56 163.83 0)
 			(hide yes)
@@
 			)
 		)
-		(property "Value" "2k6"
+		(property "Value" "2k7"
 			(at 38.1 125.7299 0)
 			(show_name no)
@@
 			)
 		)
-		(property "LCSC_PN" "C870633"
+		(property "LCSC_PN" "C2907368"
 			(at 35.56 107.95 0)
 			(hide yes)
@@
 			)
 		)
-		(property "MP" "RT1206BRD072K7L"
+		(property "MP" "FRC1206F1003TS"
 			(at 35.56 107.95 0)
 			(hide yes)
