File: Hardware/BLDC_MC_V1.0/BLDC_MC_V1.0_Connectors.kicad_sch (KiCad schematic)
At the start: 15 parts, among them J1 Conn_01x01_Pin, J2 Conn_01x01_Pin, J5 S6B-PH-K-S_LF__SN_, J6 Conn_01x01_Pin, J7 Conn_01x01_Pin, J8 S10B-PHDSS LFSN, J9 Conn_01x01_Pin

Commit message: Update board layout
Connections:
- net CAN_H renamed CAN_N
- net CAN_L renamed CAN_P
Changed lines of the file:
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@@
+	(wire
+		(pts
+			(xy 140.97 76.2) (xy 142.24 76.2)
+		)
+		(stroke
+			(width 0)
+			(type default)
+		)
+	)
 	(wire
 		(pts
@@
 	(wire
 		(pts
-			(xy 139.7 76.2) (xy 142.24 76.2)
-		)
-		(stroke
-			(width 0)
-			(type default)
-		)
-	)
-	(wire
-		(pts
 			(xy 207.01 91.44) (xy 207.01 93.98)
 		)
@@
 	(wire
 		(pts
-			(xy 139.7 78.74) (xy 142.24 78.74)
-		)
-		(stroke
-			(width 0)
-			(type default)
-		)
-	)
-	(wire
-		(pts
 			(xy 137.16 97.79) (xy 137.16 83.82)
 		)
@@
 		)
 	)
+	(wire
+		(pts
+			(xy 140.97 78.74) (xy 142.24 78.74)
+		)
+		(stroke
+			(width 0)
+			(type default)
+		)
+	)
 	(hierarchical_label "Hall_C"
 		(shape output)
@@
 		)
 	)
-	(hierarchical_label "CAN_H"
+	(hierarchical_label "CAN_P"
 		(shape bidirectional)
-		(at 139.7 76.2 180)
+		(at 140.97 78.74 180)
 		(effects
 			(font
@@
 		)
 	)
-	(hierarchical_label "CAN_L"
+	(hierarchical_label "CAN_N"
 		(shape bidirectional)
-		(at 139.7 78.74 180)
-		(effects
-			(font
+		(at 140.97 76.2 180)
+		(effects
+			(font
