File: Hardware/BLDC_MC_V1.0/BLDC_MC_V1.0_Connectors.kicad_sch (KiCad schematic)
At the start: 15 parts, among them J1 Conn_01x01_Pin, J2 Conn_01x01_Pin, J5 S6B-PH-K-S_LF__SN_, J6 Conn_01x01_Pin, J7 Conn_01x01_Pin, J8 S10B-PHDSS LFSN, J9 Conn_01x01_Pin

Commit message: Edited the label of the Schematic sheets
Other:
- company: (none) -> Ahmed Aboeita
Changed lines of the file:
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@@
 	(title_block
 		(title "${Project_Name}")
-		(date "2026-03-08")
-		(rev "V1")
+		(date "2026-08-17")
+		(rev "V1.0")
+		(company "Ahmed Aboeita")
+		(comment 1 "8-Layer High-TG180 PCB with Kelvin Current Sensing")
+		(comment 2 "Power Stage: 3-Phase Inverter with Active Reverse Polarity & E-Fuse OCP")
+		(comment 3 "Core MCU: STM32G431RBT6 (FOC & CORDIC Processing, 100 kHz PWM)")
+		(comment 4 "Stackup & Sensing: System Ratings: 100V DC Bus | 50A Continuous | T_A = 125 degrees  ")
 	)
 	(rectangle
