File: Hardware/BLDC_MC_V1.0/BLDC_MC_V1.0_CAN_Transceiver.kicad_sch (KiCad schematic)
At the start: 11 parts, among them U2 TCAN334DR

Commit message: Update board layout
Connections:
- net CANH renamed CAN_IC_P
- net CANL renamed CAN_IC_N
- net CAN_H renamed CAN_P
- net CAN_L renamed CAN_N
Changed lines of the file:
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@@
 		)
 	)
-	(label "CANH"
+	(label "CAN_IC_P"
 		(at 157.48 83.82 0)
 		(effects
 			(font
-				(size 1.27 1.27)
+				(size 1.016 1.016)
 			)
 			(justify left bottom)
@@
 		)
 	)
-	(label "CANL"
+	(label "CAN_IC_N"
 		(at 157.48 91.44 0)
 		(effects
 			(font
-				(size 1.27 1.27)
+				(size 1.016 1.016)
 			)
 			(justify left bottom)
@@
 		)
 	)
-	(hierarchical_label "CAN_H"
+	(hierarchical_label "CAN_P"
 		(shape bidirectional)
 		(at 254 78.74 0)
@@
 		)
 	)
-	(hierarchical_label "CAN_L"
+	(hierarchical_label "CAN_N"
 		(shape bidirectional)
 		(at 254 96.52 0)

Commit message: Edited the label of the Schematic sheets
Other:
- company: (none) -> Ahmed Aboeita
Changed lines of the file:
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@@
 	(title_block
 		(title "${Project_Name}")
-		(date "2026-01-05")
-		(rev "V1")
+		(date "2026-08-17")
+		(rev "V1.0")
+		(company "Ahmed Aboeita")
+		(comment 1 "8-Layer High-TG180 PCB with Kelvin Current Sensing")
+		(comment 2 "Power Stage: 3-Phase Inverter with Active Reverse Polarity & E-Fuse OCP")
+		(comment 3 "Core MCU: STM32G431RBT6 (FOC & CORDIC Processing, 100 kHz PWM)")
+		(comment 4 "Stackup & Sensing: System Ratings: 100V DC Bus | 50A Continuous | T_A = 125 degrees  ")
 	)
 	(rectangle
