File: Hardware/BLDC_MC_V1.0/BLDC_MC_V1.0.kicad_sch (KiCad schematic)
At the start: 0 parts

Commit message: Update board layout
Other:
- sheet BLDC_MC_V1.0_CAN_Transceiver ports: added CAN_N, CAN_P; removed CAN_H, CAN_L
- sheet BLDC_MC_V1.0_Connectors ports: added CAN_N, CAN_P; removed CAN_H, CAN_L
Changed lines of the file:
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@@
 			)
 		)
-		(pin "CAN_L" bidirectional
+		(pin "CAN_N" bidirectional
 			(at 45.72 105.41 180)
 			(effects
@@
 			)
 		)
-		(pin "CAN_H" bidirectional
+		(pin "CAN_P" bidirectional
 			(at 45.72 102.87 180)
 			(effects
@@
 			)
 		)
-		(pin "CAN_H" bidirectional
+		(pin "CAN_P" bidirectional
 			(at 46.99 135.89 180)
 			(effects
@@
 			)
 		)
-		(pin "CAN_L" bidirectional
+		(pin "CAN_N" bidirectional
 			(at 46.99 133.35 180)
 			(effects

Commit message: Update the silk screen of the board
Other:
- company: (none) -> Ahmed Aboeita
Changed lines of the file:
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@@
 	(title_block
 		(title "${Project_Name}")
-		(date "2026-01-05")
-		(rev "V1")
+		(date "2026-08-17")
+		(rev "V1.0")
+		(company "Ahmed Aboeita")
+		(comment 1 "8-Layer High-TG180 PCB with Kelvin Current Sensing")
+		(comment 2 "Power Stage: 3-Phase Inverter with Active Reverse Polarity & E-Fuse OCP")
+		(comment 3 "Core MCU: STM32G431RBT6 (FOC & CORDIC Processing, 100 kHz PWM)")
+		(comment 4 "Stackup & Sensing: System Ratings: 100V DC Bus | 50A Continuous | T_A = 125 degrees  ")
 	)
 	(text "Inverter\nbridge"
